File: jack_pcb/jack_pcb.sch (KiCad schematic (older format))
At the start: 89 parts, among them J0 PJ301M-12, J1 PJ301M-12, J10 PJ301M-12, J101 RJ45, J102 RJ45, J103 RJ45, J104 RJ45, J105 RJ45, J106 RJ45, J107 RJ45, J108 RJ45, J11 PJ301M-12, J110 Conn_02x16_Odd_Even, J111 Conn_02x25_Odd_Even, J12 PJ301M-12, J13 PJ301M-12, J14 PJ301M-12, J15 PJ301M-12, J16 PJ301M-12, J17 PJ301M-12, J18 PJ301M-12, J19 PJ301M-12, J2 PJ301M-12, J20 PJ301M-12, J21 PJ301M-12, J22 PJ301M-12, J23 PJ301M-12, J24 PJ301M-12, J25 PJ301M-12, J26 PJ301M-12, J27 PJ301M-12, J28 PJ301M-12, J29 PJ301M-12, J3 PJ301M-12, J30 PJ301M-12, J31 PJ301M-12, J32 DIN-5, J33 DIN-5, J34 DIN-5, J4 PJ301M-12, J5 PJ301M-12, J6 PJ301M-12, J7 PJ301M-12, J8 PJ301M-12, J9 PJ301M-12, U1 74HC14, U5 6N138

Commit message: finalized jack board
Parts:
- removed C?: .1uF, Capacitor_THT:C_Axial_L3.8mm_D2.6mm_P7.50mm_Horizontal, symbol Device:C_Small
- removed J111: Conn_02x25_Odd_Even, Connector_PinSocket_2.54mm:PinSocket_2x25_P2.54mm_Vertical, symbol Connector_Generic:Conn_02x25_Odd_Even
- removed R1, R10, R11, R12, R13, R14, R15, R16, R17, R18, R19, R2, R20, R21, R22, R23, R24, R25, R26, R27, R28, R29, R3, R30, R37, R38, R4, R5, R6, R7, R8, R9: 1000, Resistor_THT:R_Axial_DIN0207_L6.3mm_D2.5mm_P10.16mm_Horizontal, symbol Device:R_Small_US
- added C3, C5: .1uF, Capacitor_THT:C_Axial_L3.8mm_D2.6mm_P7.50mm_Horizontal, symbol Device:C_Small
- added C4, C6: 10uF Tantalum, Capacitor_THT:C_Axial_L3.8mm_D2.6mm_P7.50mm_Horizontal, symbol Device:C_Small
- added J26: Conn_02x25_Odd_Even, Connector_PinSocket_2.54mm:PinSocket_2x25_P2.54mm_Vertical, symbol Connector_Generic:Conn_02x25_Odd_Even
- added unit 7 of U1
- gave numbers to parts that had none: 1
- renumbered C1 to C2, J7 to J1, J15 to J10, J8 to J11, J9 to J12, J10 to J13, J11 to J14, J12 to J15, J13 to J16, J14 to J17, J23 to J18, J16 to J19, J0 to J2, J17 to J20, J18 to J21, J19 to J22, J20 to J23, J21 to J24, J22 to J25, J31 to J27, J24 to J28, J25 to J29, J1 to J3, J26 to J30, J27 to J31, J28 to J32, J29 to J33, J30 to J34, J33 to J35, J34 to J36, J32 to J37, J105 to J38, J107 to J39, J2 to J4, J101 to J40, J103 to J41, J106 to J42, J108 to J43, J102 to J44, J104 to J45, J3 to J5, J4 to J6, J5 to J7, J6 to J8, J110 to J9, R31 to R1, R32 to R2, R33 to R3, R34 to R4, R35 to R5, R36 to R6, U5 to U2
Connections:
- net +12V: now also J42.7, J42.8, C3.1, C4.1; no longer J39.7, J39.8
- net +3V3: now also C5.1, C6.1
- net +5V: now also J39.7, J39.8, J43.7, J43.8, U1.14 (VCC); no longer J42.7, J42.8
- net GND: now also C3.2, C4.2, C5.2, C6.2, J26.41 (Pin_41), J26.42 (Pin_42), J26.43 (Pin_43), J26.44 (Pin_44), J26.45 (Pin_45), J26.46 (Pin_46), J26.47 (Pin_47), J26.48 (Pin_48), J26.49 (Pin_49), J26.50 (Pin_50), U1.7 (GND)
- new net VDAC0: J26.1 (Pin_1)
- new net VDAC1: J26.2 (Pin_2)
- new net VDAC10: J26.11 (Pin_11)
- new net VDAC11: J26.12 (Pin_12)
- new net VDAC12: J26.13 (Pin_13)
- new net VDAC13: J26.14 (Pin_14)
- new net VDAC14: J26.15 (Pin_15)
- new net VDAC15: J26.16 (Pin_16)
- new net VDAC16: J26.17 (Pin_17)
- new net VDAC17: J26.18 (Pin_18)
- new net VDAC18: J26.19 (Pin_19)
- new net VDAC19: J26.20 (Pin_20)
- new net VDAC2: J26.3 (Pin_3)
- new net VDAC20: J26.21 (Pin_21)
- new net VDAC21: J26.22 (Pin_22)
- new net VDAC22: J26.23 (Pin_23)
- new net VDAC23: J26.24 (Pin_24)
- new net VDAC24: J26.25 (Pin_25)
- new net VDAC25: J26.26 (Pin_26)
- new net VDAC26: J26.27 (Pin_27)
- new net VDAC27: J26.28 (Pin_28)
- new net VDAC28: J26.29 (Pin_29)
- new net VDAC29: J26.30 (Pin_30)
- new net VDAC3: J26.4 (Pin_4)
- new net VDAC30: J26.31 (Pin_31)
- new net VDAC31: J26.32 (Pin_32)
- new net VDAC4: J26.5 (Pin_5)
- new net VDAC5: J26.6 (Pin_6)
- new net VDAC6: J26.7 (Pin_7)
- new net VDAC7: J26.8 (Pin_8)
- new net VDAC8: J26.9 (Pin_9)
- new net VDAC9: J26.10 (Pin_10)
Other:
- moved on the sheet: C1, C2
