File: jack_pcb/jack_pcb.kicad_pcb (KiCad board)
At the start: 2 copper layers, 200 x 127.5 mm, 97 parts, among them J0 PJ301M-12, J1 PJ301M-12, J10 PJ301M-12, J101 RJ45, J102 RJ45, J103 RJ45, J104 RJ45, J105 RJ45, J106 RJ45, J107 RJ45, J108 RJ45, J11 PJ301M-12, J110 Conn_02x16_Odd_Even, J111 Conn_02x25_Odd_Even, J12 PJ301M-12, J13 PJ301M-12, J14 PJ301M-12, J15 PJ301M-12, J16 PJ301M-12, J17 PJ301M-12, J18 PJ301M-12, J19 PJ301M-12, J2 PJ301M-12, J20 PJ301M-12, J21 PJ301M-12, J22 PJ301M-12, J23 PJ301M-12, J24 PJ301M-12, J25 PJ301M-12, J26 PJ301M-12, J27 PJ301M-12, J28 PJ301M-12, J29 PJ301M-12, J3 PJ301M-12, J30 PJ301M-12, J31 PJ301M-12, J32 DIN-5, J33 DIN-5, J34 DIN-5, J35 USB_B, J4 PJ301M-12, J5 PJ301M-12, J6 PJ301M-12, J7 PJ301M-12, J8 PJ301M-12, J9 PJ301M-12, U1 74HC14, U10 Teensy4.1, U5 6N138, U6 74125, U7 74125, U8 74125, U9 74125

Commit message: jack board modifications
Parts:
- added REF**: MountingHole_5.3mm_M5_Pad, MountingHole:MountingHole_5.3mm_M5_Pad, F.Cu at (138.4, 160.1)
- added REF**: MountingHole_5.3mm_M5_Pad, MountingHole:MountingHole_5.3mm_M5_Pad, F.Cu at (146.4, 38.1)
Changed lines of the file:
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@@
   (general
     (thickness 1.6)
-    (drawings 7)
+    (drawings 8)
     (tracks 724)
     (zones 0)
-    (modules 97)
+    (modules 99)
     (nets 228)
   )
@@
   )
   (setup
-    (last_trace_width 0.254)
+    (last_trace_width 0.25)
     (user_trace_width 0.254)
     (user_trace_width 0.381)
@@
   )
   (module MountingHole:MountingHole_5.3mm_M5_Pad (layer F.Cu)
+    (at 138.400444 160.13619)
+    (descr "Mounting Hole 5.3mm, M5")
+    (tags "mounting hole 5.3mm m5")
+    (attr virtual)
+    (fp_text reference REF** (at 0 -6.3) (layer F.SilkS)
+      (effects (font (size 1 1) (thickness 0.15)))
+    )
+    (fp_text value MountingHole_5.3mm_M5_Pad (at 0 6.3) (layer F.Fab)
+      (effects (font (size 1 1) (thickness 0.15)))
+    )
+    (fp_text user %R (at 0.3 0) (layer F.Fab)
+      (effects (font (size 1 1) (thickness 0.15)))
+    )
+    (fp_circle (center 0 0) (end 5.3 0) (layer Cmts.User) (width 0.15))
+    (fp_circle (center 0 0) (end 5.55 0) (layer F.CrtYd) (width 0.05))
+    (pad 1 thru_hole circle (at 0 0) (size 10.6 10.6) (drill 5.3) (layers *.Cu *.Mask))
+  )
+  (module MountingHole:MountingHole_5.3mm_M5_Pad (layer F.Cu)
+    (at 146.400444 38.13619)
+    (descr "Mounting Hole 5.3mm, M5")
+    (tags "mounting hole 5.3mm m5")
+    (attr virtual)
+    (fp_text reference REF** (at 0 -6.3) (layer F.SilkS)
+      (effects (font (size 1 1) (thickness 0.15)))
+    )
+    (fp_text value MountingHole_5.3mm_M5_Pad (at 0 6.3) (layer F.Fab)
+      (effects (font (size 1 1) (thickness 0.15)))
+    )
+    (fp_text user %R (at 0.3 0) (layer F.Fab)
+      (effects (font (size 1 1) (thickness 0.15)))
+    )
+    (fp_circle (center 0 0) (end 5.3 0) (layer Cmts.User) (width 0.15))
+    (fp_circle (center 0 0) (end 5.55 0) (layer F.CrtYd) (width 0.05))
+    (pad 1 thru_hole circle (at 0 0) (size 10.6 10.6) (drill 5.3) (layers *.Cu *.Mask))
+  )
+  (module MountingHole:MountingHole_5.3mm_M5_Pad (layer F.Cu)
     (at 235.900444 38.63619)
     (descr "Mounting Hole 5.3mm, M5")
@@
     )
   )
+  (dimension 200.500623 (width 0.12) (layer F.SilkS)
+    (gr_text "7.8937 in" (at 142.819236 4.986403 359.8571181) (layer F.SilkS)
+      (effects (font (size 1 1) (thickness 0.15)))
+    )
+    (feature1 (pts (xy 243 33) (xy 243.067531 5.91998)))
+    (feature2 (pts (xy 42.5 32.5) (xy 42.567531 5.41998)))
+    (crossbar (pts (xy 42.566069 6.006399) (xy 243.066069 6.506399)))
+    (arrow1a (pts (xy 243.066069 6.506399) (xy 241.938106 7.090009)))
+    (arrow1b (pts (xy 243.066069 6.506399) (xy 241.941031 5.917171)))
+    (arrow2a (pts (xy 42.566069 6.006399) (xy 43.691107 6.595627)))
+    (arrow2b (pts (xy 42.566069 6.006399) (xy 43.694032 5.422789)))
+  )
   (gr_line (start 242.5 160) (end 242.5 155) (layer Edge.Cuts) (width 0.05))

Commit message: finalized jack board
Parts:
- removed J107: RJ45, Connector_RJ:RJ45_Amphenol_54602-x08_Horizontal
- removed J111: Conn_02x25_Odd_Even, Connector_PinSocket_2.54mm:PinSocket_2x25_P2.54mm_Vertical
- removed the R1 at (58.5, 60.0)
- removed the R2 at (55.0, 60.0)
- removed the R3 at (88.7, 60.0)
- removed the R4 at (83.7, 60.0)
- removed the R5 at (118.7, 60.0)
- removed the R6 at (113.7, 60.0)
- removed the REF** at (138.4, 160.1)
- removed the REF** at (146.4, 38.1)
- removed the REF** at (235.9, 38.6)
- removed the REF** at (56.2, 38.6)
- removed the REF** at (48.9, 153.4)
- removed the REF** at (235.0, 152.5)
- removed U10: Teensy4.1, teensy2:Teensy41
- added C10: .1uF, Capacitor_THT:C_Axial_L3.8mm_D2.6mm_P7.50mm_Horizontal, B.Cu at (101.0, 46.1)
- added C11: .1uF, Capacitor_THT:C_Axial_L3.8mm_D2.6mm_P7.50mm_Horizontal, B.Cu at (116.0, 46.0)
- added C12: .1uF, Capacitor_THT:C_Axial_L3.8mm_D2.6mm_P7.50mm_Horizontal, B.Cu at (131.0, 46.0)
- added C13: .1uF, Capacitor_THT:C_Axial_L3.8mm_D2.6mm_P7.50mm_Horizontal, B.Cu at (146.0, 46.0)
- added C14: .1uF, Capacitor_THT:C_Axial_L3.8mm_D2.6mm_P7.50mm_Horizontal, B.Cu at (161.0, 46.0)
- added C15: .1uF, Capacitor_THT:C_Axial_L3.8mm_D2.6mm_P7.50mm_Horizontal, B.Cu at (56.0, 66.5)
- added C16: .1uF, Capacitor_THT:C_Axial_L3.8mm_D2.6mm_P7.50mm_Horizontal, B.Cu at (71.0, 66.0)
- added C17: .1uF, Capacitor_THT:C_Axial_L3.8mm_D2.6mm_P7.50mm_Horizontal, B.Cu at (86.0, 66.5)
- added C18: .1uF, Capacitor_THT:C_Axial_L3.8mm_D2.6mm_P7.50mm_Horizontal, B.Cu at (101.0, 66.5)
- added C19: .1uF, Capacitor_THT:C_Axial_L3.8mm_D2.6mm_P7.50mm_Horizontal, B.Cu at (116.0, 66.0)
- added C2: 10uF Tantalum, Capacitor_THT:C_Axial_L3.8mm_D2.6mm_P7.50mm_Horizontal, B.Cu at (193.3, 62.5)
- added C20: .1uF, Capacitor_THT:C_Axial_L3.8mm_D2.6mm_P7.50mm_Horizontal, B.Cu at (131.0, 66.5)
- added C21: .1uF, Capacitor_THT:C_Axial_L3.8mm_D2.6mm_P7.50mm_Horizontal, B.Cu at (146.0, 67.0)
- added C22: .1uF, Capacitor_THT:C_Axial_L3.8mm_D2.6mm_P7.50mm_Horizontal, B.Cu at (161.0, 66.0)
- added C23: .1uF, Capacitor_THT:C_Axial_L3.8mm_D2.6mm_P7.50mm_Horizontal, B.Cu at (56.0, 86.0)
- added C24: .1uF, Capacitor_THT:C_Axial_L3.8mm_D2.6mm_P7.50mm_Horizontal, B.Cu at (56.0, 106.0)
- added C25: .1uF, Capacitor_THT:C_Axial_L3.8mm_D2.6mm_P7.50mm_Horizontal, B.Cu at (71.0, 105.5)
- added C26: .1uF, Capacitor_THT:C_Axial_L3.8mm_D2.6mm_P7.50mm_Horizontal, B.Cu at (86.0, 106.5)
- added C27: .1uF, Capacitor_THT:C_Axial_L3.8mm_D2.6mm_P7.50mm_Horizontal, B.Cu at (101.0, 106.5)
- added C28: .1uF, Capacitor_THT:C_Axial_L3.8mm_D2.6mm_P7.50mm_Horizontal, B.Cu at (116.0, 107.0)
- added C29: .1uF, Capacitor_THT:C_Axial_L3.8mm_D2.6mm_P7.50mm_Horizontal, B.Cu at (131.0, 106.5)
- added C3: .1uF, Capacitor_THT:C_Axial_L3.8mm_D2.6mm_P7.50mm_Horizontal, B.Cu at (193.3, 70.7)
- added C30: .1uF, Capacitor_THT:C_Axial_L3.8mm_D2.6mm_P7.50mm_Horizontal, B.Cu at (146.0, 106.0)
- added C31: .1uF, Capacitor_THT:C_Axial_L3.8mm_D2.6mm_P7.50mm_Horizontal, B.Cu at (161.0, 106.0)
- added C32: .1uF, Capacitor_THT:C_Axial_L3.8mm_D2.6mm_P7.50mm_Horizontal, B.Cu at (71.0, 86.0)
- added C33: .1uF, Capacitor_THT:C_Axial_L3.8mm_D2.6mm_P7.50mm_Horizontal, B.Cu at (86.0, 87.0)
- added C34: .1uF, Capacitor_THT:C_Axial_L3.8mm_D2.6mm_P7.50mm_Horizontal, B.Cu at (101.0, 86.5)
- added C35: .1uF, Capacitor_THT:C_Axial_L3.8mm_D2.6mm_P7.50mm_Horizontal, B.Cu at (116.0, 86.0)
- added C36: .1uF, Capacitor_THT:C_Axial_L3.8mm_D2.6mm_P7.50mm_Horizontal, B.Cu at (131.0, 86.0)
- added C37: .1uF, Capacitor_THT:C_Axial_L3.8mm_D2.6mm_P7.50mm_Horizontal, B.Cu at (146.0, 86.0)
- added C38: .1uF, Capacitor_THT:C_Axial_L3.8mm_D2.6mm_P7.50mm_Horizontal, B.Cu at (161.0, 86.5)
- added C4: 10uF Tantalum, Capacitor_THT:C_Axial_L3.8mm_D2.6mm_P7.50mm_Horizontal, B.Cu at (193.3, 66.6)
- added C5: .1uF, Capacitor_THT:C_Axial_L3.8mm_D2.6mm_P7.50mm_Horizontal, B.Cu at (193.3, 54.3)
- added C6: 10uF Tantalum, Capacitor_THT:C_Axial_L3.8mm_D2.6mm_P7.50mm_Horizontal, B.Cu at (193.3, 50.2)
- added C7: .1uF, Capacitor_THT:C_Axial_L3.8mm_D2.6mm_P7.50mm_Horizontal, B.Cu at (71.0, 46.0)
- added C8: .1uF, Capacitor_THT:C_Axial_L3.8mm_D2.6mm_P7.50mm_Horizontal, B.Cu at (56.0, 46.0)
- added C9: .1uF, Capacitor_THT:C_Axial_L3.8mm_D2.6mm_P7.50mm_Horizontal, B.Cu at (86.0, 46.5)
- added J26: Conn_02x25_Odd_Even, Connector_PinSocket_2.54mm:PinSocket_2x25_P2.54mm_Vertical, B.Cu at (171.0, 47.4)
- added J39: RJ45, Connector_RJ:RJ45_Amphenol_54602-x08_Horizontal, F.Cu at (208.7, 142.1)
- added J47: Conn_01x24, Connector_PinHeader_2.54mm:PinHeader_1x24_P2.54mm_Vertical, B.Cu at (130.1, 148.9)
- added J48: Conn_01x24, Connector_PinHeader_2.54mm:PinHeader_1x24_P2.54mm_Vertical, B.Cu at (130.1, 124.9)
- added R31: 1000, Resistor_THT:R_Axial_DIN0207_L6.3mm_D2.5mm_P10.16mm_Horizontal, B.Cu at (149.0, 120.0)
- added R32: 1000, Resistor_THT:R_Axial_DIN0207_L6.3mm_D2.5mm_P10.16mm_Horizontal, B.Cu at (59.0, 100.0)
- added R33: 1000, Resistor_THT:R_Axial_DIN0207_L6.3mm_D2.5mm_P10.16mm_Horizontal, B.Cu at (74.0, 100.0)
- added R34: 1000, Resistor_THT:R_Axial_DIN0207_L6.3mm_D2.5mm_P10.16mm_Horizontal, B.Cu at (88.5, 100.0)
- added R35: 1000, Resistor_THT:R_Axial_DIN0207_L6.3mm_D2.5mm_P10.16mm_Horizontal, B.Cu at (103.0, 100.0)
- added R36: 1000, Resistor_THT:R_Axial_DIN0207_L6.3mm_D2.5mm_P10.16mm_Horizontal, B.Cu at (118.0, 100.0)
- added REF**: MountingHole_4.3mm_M4_DIN965_Pad, MountingHole:MountingHole_4.3mm_M4_DIN965_Pad, F.Cu at (147.0, 138.7)
- added REF**: MountingHole_4.3mm_M4_DIN965_Pad, MountingHole:MountingHole_4.3mm_M4_DIN965_Pad, F.Cu at (238.2, 155.6)
- added REF**: MountingHole_4.3mm_M4_DIN965_Pad, MountingHole:MountingHole_4.3mm_M4_DIN965_Pad, F.Cu at (47.4, 154.7)
- added REF**: MountingHole_4.3mm_M4_DIN965_Pad, MountingHole:MountingHole_4.3mm_M4_DIN965_Pad, F.Cu at (164.1, 37.0)
- added REF**: MountingHole_4.3mm_M4_DIN965_Pad, MountingHole:MountingHole_4.3mm_M4_DIN965_Pad, F.Cu at (47.2, 36.9)
- added REF**: MountingHole_4.3mm_M4_DIN965_Pad, MountingHole:MountingHole_4.3mm_M4_DIN965_Pad, F.Cu at (237.4, 36.9)
- added U7: Teensy4.1, teensy2:Teensy41, B.Cu at (101.1, 136.9)
- moved J46 173.0 mm to (57.0, 142.0), turned to 270 degrees
- moved U6 165.3 mm to (223.2, 122.4)
- moved U4 113.1 mm to (223.2, 111.4), turned to 270 degrees
- moved U5 109.0 mm to (202.0, 125.0), turned to 270 degrees
- moved R24 101.5 mm to (44.1, 120.0), turned to 0 degrees
- moved R7 94.5 mm to (54.2, 59.9), turned to 180 degrees
- moved C1 91.1 mm to (193.3, 58.4)
- moved R8 85.2 mm to (58.5, 59.8), turned to 0 degrees
- moved R16 84.7 mm to (59.0, 80.0), turned to 0 degrees
- moved R37 77.9 mm to (134.0, 100.0)
- moved U3 73.9 mm to (202.0, 114.0), turned to 270 degrees
- moved R6 44.5 mm to (194.0, 142.0)
- moved R22 40.7 mm to (149.0, 80.0), turned to 0 degrees
- moved R12 40.6 mm to (119.0, 60.0), turned to 0 degrees
- moved R14 40.6 mm to (149.0, 60.0), turned to 0 degrees
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- renumbered J7 to J1, J15 to J10, J8 to J11, J9 to J12, J10 to J13, J11 to J14, J12 to J15, J13 to J16, J14 to J17, J23 to J18, J16 to J19, J0 to J2, J17 to J20, J18 to J21, J19 to J22, J20 to J23, J21 to J24, J22 to J25, J31 to J27, J24 to J28, J25 to J29, J1 to J3, J26 to J30, J27 to J31, J28 to J32, J29 to J33, J30 to J34, J33 to J35, J34 to J36, J32 to J37, J105 to J38, J2 to J4, J101 to J40, J103 to J41, J106 to J42, J108 to J43, J102 to J44, J104 to J45, J35 to J46, J3 to J5, J4 to J6, J5 to J7, J6 to J8, J110 to J9, R31 to R1, R32 to R2, R33 to R3, R34 to R4, R35 to R5, R36 to R6, U5 to U2, U6 to U3, U7 to U4, U8 to U5, U9 to U6
Connections:
- J42 pad 7: +5V -> +12V
- J42 pad 8: +5V -> +12V
- J43 pad 7: Net-(J108-Pad7) -> +5V
- J43 pad 8: Net-(J108-Pad7) -> +5V
- R10 pad 1: Net-(J111-Pad9) -> V3
- R10 pad 2: V8 -> VDAC3
- R11 pad 1: V13 -> V4
- R11 pad 2: Net-(J111-Pad14) -> VDAC4
- R12 pad 1: Net-(J111-Pad11) -> V5
- R12 pad 2: V10 -> VDAC5
- R13 pad 1: V15 -> V6
- R13 pad 2: Net-(J111-Pad16) -> VDAC6
- R14 pad 1: Net-(J111-Pad13) -> V7
- R14 pad 2: V12 -> VDAC7
- R15 pad 1: V17 -> V8
- R15 pad 2: Net-(J111-Pad18) -> VDAC8
- R16 pad 1: Net-(J111-Pad15) -> V9
- R16 pad 2: V14 -> VDAC9
- R17 pad 1: V19 -> V10
- R17 pad 2: Net-(J111-Pad20) -> VDAC10
- R18 pad 1: Net-(J111-Pad17) -> V11
- R18 pad 2: V16 -> VDAC11
- R19 pad 1: V21 -> V12
- R19 pad 2: Net-(J111-Pad22) -> VDAC12
- R20 pad 1: Net-(J111-Pad19) -> V13
- R20 pad 2: V18 -> VDAC13
- R21 pad 1: V23 -> V14
- R21 pad 2: Net-(J111-Pad24) -> VDAC14
- R22 pad 1: Net-(J111-Pad21) -> V15
- R22 pad 2: V20 -> VDAC15
- R23 pad 1: V25 -> V16
- R23 pad 2: Net-(J111-Pad26) -> VDAC16
- R24 pad 1: Net-(J111-Pad23) -> V24
- R24 pad 2: V22 -> VDAC24
- R25 pad 1: V27 -> V25
- R25 pad 2: Net-(J111-Pad28) -> VDAC25
- R26 pad 1: Net-(J111-Pad25) -> V26
- R26 pad 2: V24 -> VDAC26
- R27 pad 1: V29 -> V27
- R27 pad 2: Net-(J111-Pad30) -> VDAC27
- R28 pad 1: Net-(J111-Pad27) -> V28
- R28 pad 2: V26 -> VDAC28
- R29 pad 1: V31 -> V29
- R29 pad 2: Net-(J111-Pad32) -> VDAC29
- R30 pad 1: Net-(J111-Pad29) -> V30
- R30 pad 2: V28 -> VDAC30
- R37 pad 1: V9 -> V22
- R37 pad 2: Net-(J111-Pad10) -> VDAC22
- R38 pad 1: Net-(J111-Pad31) -> V23
- R38 pad 2: V30 -> VDAC23
- R7 pad 1: V7 -> VDAC0
- R7 pad 2: Net-(J111-Pad8) -> V0
- R8 pad 1: Net-(J111-Pad7) -> V1
- R8 pad 2: V6 -> VDAC1
- R9 pad 1: V11 -> V2
- R9 pad 2: Net-(J111-Pad12) -> VDAC2
- U1 pad 14: (no net) -> +5V
- U1 pad 7: (no net) -> GND
- U3 pad 11: MOTOR4 -> MOTOR2
- U3 pad 12: PWMOUT4 -> PWMOUT2
- U3 pad 14: VCC -> +5V
- U3 pad 5: PWMOUT2 -> PWMOUT3
- U3 pad 6: MOTOR2 -> MOTOR3
- U3 pad 8: MOTOR3 -> MOTOR4
- U3 pad 9: PWMOUT3 -> PWMOUT4
- U4 pad 11: MOTOR8 -> MOTOR6
- U4 pad 12: PWMOUT8 -> PWMOUT6
- U4 pad 14: VCC -> +5V
- U4 pad 5: PWMOUT6 -> PWMOUT7
- U4 pad 6: MOTOR6 -> MOTOR7
- U4 pad 8: MOTOR7 -> MOTOR8
- U4 pad 9: PWMOUT7 -> PWMOUT8
- U5 pad 11: LED4 -> LED2
- U5 pad 12: LEDOUT4 -> LEDOUT2
- U5 pad 14: VCC -> +5V
- U5 pad 5: LEDOUT2 -> LEDOUT3
- U5 pad 6: LED2 -> LED3
- U5 pad 8: LED3 -> LED4
- U5 pad 9: LEDOUT3 -> LEDOUT4
- U6 pad 11: LED8 -> LED6
- U6 pad 12: LEDOUT8 -> LEDOUT6
- U6 pad 14: VCC -> +5V
- U6 pad 5: LEDOUT6 -> LEDOUT7
- U6 pad 6: LED6 -> LED7
- U6 pad 8: LED7 -> LED8
- U6 pad 9: LEDOUT7 -> LEDOUT8
Routing:
- net LED6: track 326.8 -> 4.01 mm, vias 2 -> 0
- net LED7: track 321.9 -> 15.8 mm
- net LED3: track 211.9 -> 18.3 mm, vias 1 -> 0
- net Net-(J111-Pad25): track 192.4 -> 0.00 mm
- net LED8: track 198.6 -> 7.05 mm
- net LED5: track 202.4 -> 14.6 mm
- net +5V: track 211.5 -> 397.8 mm, vias 0 -> 1
- net MOTOR6: track 210.3 -> 26.9 mm
- net PWMOUT8: track 9.40 -> 179.7 mm, vias 0 -> 1
- net LEDOUT8: track 49.9 -> 210.3 mm, vias 0 -> 2
- net LEDOUT6: track 26.2 -> 182.9 mm, vias 0 -> 1
- net LEDOUT4: track 9.62 -> 164.2 mm, vias 0 -> 1
- net VDAC24: track 0.00 -> 152.0 mm
- net MOTOR1: track 168.6 -> 19.4 mm
- net PWMOUT7: track 20.4 -> 165.2 mm, vias 0 -> 1
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- added copper zone on F.Cu, net GND
- removed copper zone on B.Cu, net GND
Other:
- outline, holes or cut-outs redrawn
- board text added: "12V"
- board text added: "3.3V"
- board text added: "5V"
- board text added: "GND"
- board text added: "IN1"
- board text added: "IN1-4"
- board text added: "IN13-16"
- board text added: "IN16"
- board text added: "IN5-8"
- board text added: "IN9-12"
- board text added: "LED OUT (1 - 4)"
- board text added: "LED OUT (5 - 8)"
- board text added: "MIDI INPUT"
- board text added: "MIDI OUTPUT"
- board text added: "MIDI+"
- board text added: "MIDI-"
- board text added: "MIDI_OUT"
- board text added: "MIDI_THRU"
- board text added: "MOTOR (PWM 1-4)"
- board text added: "MOTOR (PWM 5-8)"
- board text added: "V0"
- board text added: "V1"
- board text added: "V16"
- board text added: "V2"
- board text added: "V24"
- board text added: "V3"
- board text added: "V30"
- board text added: "V31"
- board text added: "V4"
- board text added: "V5"
- board text added: "V6"
- board text added: "V7"
- board text added: "V8"
- board text added: "connector to Central PCB"
- board text added: "connector to DAC"

Commit message: gerbers and small finalizations to boards
Other:
- board text added: "Harmonic Content Jack and Visual PCB Rev. 1 October 2021"
Changed lines of the file:
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@@
   (general
     (thickness 1.6)
-    (drawings 58)
+    (drawings 61)
     (tracks 1157)
     (zones 0)
@@
   (page A4)
   (layers
-    (0 F.Cu signal)
+    (0 F.Cu signal hide)
     (31 B.Cu signal)
     (32 B.Adhes user)
@@
   )
   (setup
-    (last_trace_width 0.762)
+    (last_trace_width 0.25)
     (user_trace_width 0.254)
     (user_trace_width 0.381)
@@
     (pcbplotparams
       (layerselection 0x010fc_ffffffff)
-      (usegerberextensions false)
+      (usegerberextensions true)
       (usegerberattributes false)
       (usegerberadvancedattributes false)
@@
       (outputformat 1)
       (mirror false)
-      (drillshape 1)
+      (drillshape 0)
       (scaleselection 1)
-      (outputdirectory ""))
+      (outputdirectory "jackpcb_gerbers"))
   )
   (net 0 "")
@@
     )
   )
+  (dimension 127.5 (width 0.15) (layer Dwgs.User)
+    (gr_text "5.0197 in" (at 252.8 96.25 270) (layer Dwgs.User)
+      (effects (font (size 1 1) (thickness 0.15)))
+    )
+    (feature1 (pts (xy 242.5 160) (xy 252.086421 160)))
+    (feature2 (pts (xy 242.5 32.5) (xy 252.086421 32.5)))
+    (crossbar (pts (xy 251.5 32.5) (xy 251.5 160)))
+    (arrow1a (pts (xy 251.5 160) (xy 250.913579 158.873496)))
+    (arrow1b (pts (xy 251.5 160) (xy 252.086421 158.873496)))
+    (arrow2a (pts (xy 251.5 32.5) (xy 250.913579 33.626504)))
+    (arrow2b (pts (xy 251.5 32.5) (xy 252.086421 33.626504)))
+  )
+  (dimension 200 (width 0.15) (layer Dwgs.User)
+    (gr_text "7.8740 in" (at 142.5 2.9) (layer Dwgs.User)
+      (effects (font (size 1 1) (thickness 0.15)))
+    )
+    (feature1 (pts (xy 242.5 32.5) (xy 242.5 3.613579)))
+    (feature2 (pts (xy 42.5 32.5) (xy 42.5 3.613579)))
+    (crossbar (pts (xy 42.5 4.2) (xy 242.5 4.2)))
+    (arrow1a (pts (xy 242.5 4.2) (xy 241.373496 4.786421)))
+    (arrow1b (pts (xy 242.5 4.2) (xy 241.373496 3.613579)))
+    (arrow2a (pts (xy 42.5 4.2) (xy 43.626504 4.786421)))
+    (arrow2b (pts (xy 42.5 4.2) (xy 43.626504 3.613579)))
+  )
+  (gr_text "Harmonic Content \nJack and Visual PCB\nRev. 1\nOctober 2021" (at 187.2 39.8) (layer F.SilkS)
+    (effects (font (size 1.7 1.7) (thickness 0.425) italic))
+  )
+  (gr_text "Harmonic Content \nJack and Visual PCB\nRev. 1\nOctober 2021" (at 182 116.9) (layer B.SilkS)
+    (effects (font (size 1.7 1.7) (thickness 0.425) italic) (justify mirror))
+  )
   (gr_text V24 (at 49 102.4) (layer F.SilkS)
     (effects (font (size 1 1) (thickness 0.15)))
@@
     (effects (font (size 0.8128 0.8128) (thickness 0.1524)) (justify mirror))
   )
-  (gr_text "LED OUT (5 - 8)" (at 232.4 157.8) (layer F.SilkS)
+  (gr_text "LED OUT (5 - 8)" (at 228.2 152.3) (layer F.SilkS)
     (effects (font (size 1 1) (thickness 0.15)))
   )
@@
   (gr_line (start 242.5 160) (end 46.2 160) (layer Edge.Cuts) (width 0.05))
   (gr_line (start 46.2 160) (end 42.5 160) (layer Edge.Cuts) (width 0.05))
-  (dimension 127.5 (width 0.12) (layer F.SilkS)
-    (gr_text "5.0197 in" (at 284.27 96.25 270) (layer F.SilkS)
-      (effects (font (size 1 1) (thickness 0.15)))
-    )
-    (feature1 (pts (xy 242.5 160) (xy 283.586421 160)))
-    (feature2 (pts (xy 242.5 32.5) (xy 283.586421 32.5)))
-    (crossbar (pts (xy 283 32.5) (xy 283 160)))
-    (arrow1a (pts (xy 283 160) (xy 282.413579 158.873496)))
-    (arrow1b (pts (xy 283 160) (xy 283.586421 158.873496)))
-    (arrow2a (pts (xy 283 32.5) (xy 282.413579 33.626504)))
-    (arrow2b (pts (xy 283 32.5) (xy 283.586421 33.626504)))
-  )
   (gr_line (start 242.5 160) (end 242.5 155) (layer Edge.Cuts) (width 0.05))
   (gr_line (start 42.5 155) (end 42.5 160) (layer Edge.Cuts) (width 0.05))
@@
   (segment (start 217.24 120.48863) (end 215.890501 119.139131) (width 0.381) (layer B.Cu) (net 90))
   (segment (start 214 101.035942) (end 214 93.1) (width 0.381) (layer B.Cu) (net 90))
-  (segment (start 209.62 121.62) (end 210.810501 120.429499) (width 0.381) (layer B.Cu) (net 92))
   (segment (start 214.7 112.86863) (end 211.6 109.76863) (width 0.381) (layer B.Cu) (net 91))
   (segment (start 214.7 114) (end 214.7 112.86863) (width 0.381) (layer B.Cu) (net 91))
   (segment (start 211.6 109.76863) (end 211.6 96.8) (width 0.381) (layer B.Cu) (net 91))
   (segment (start 211.6 96.8) (end 212.6 95.8) (width 0.381) (layer B.Cu) (net 91))
+  (segment (start 209.62 121.62) (end 210.810501 120.429499) (width 0.381) (layer B.Cu) (net 92))
   (segment (start 211.6 93.4) (end 211.4 93.2) (width 0.381) (layer B.Cu) (net 92))
   (segment (start 210.810501 96.717441) (end 211.5 96.027942) (width 0.381) (layer B.Cu) (net 92))
@@
   (segment (start 230.82 130.02) (end 230.82 131.15137) (width 0.381) (layer B.Cu) (net 104))
   (segment (start 230.5 131.47137) (end 230.5 133.9) (width 0.381) (layer B.Cu) (net 104))
+  (segment (start 229.409499 133.362559) (end 229.409499 136.309499) (width 0.381) (layer B.Cu) (net 105))
+  (segment (start 229.5 133.272058) (end 229.409499 133.362559) (width 0.381) (layer B.Cu) (net 105))
+  (segment (start 229.5 124.75137) (end 229.5 133.272058) (width 0.381) (layer B.Cu) (net 105))
+  (segment (start 228.28 122.4) (end 228.28 123.53137) (width 0.381) (layer B.Cu) (net 105))
+  (segment (start 228.28 123.53137) (end 229.5 124.75137) (width 0.381) (layer B.Cu) (net 105))
+  (segment (start 229.409499 136.309499) (end 229.5 136.4) (width 0.381) (layer B.Cu) (net 105))
   (segment (start 159.00951 140.40949) (end 165.10949 140.40949) (width 0.381) (layer B.Cu) (net 106))
   (segment (start 159 142) (end 159 140.419) (width 0.381) (layer B.Cu) (net 106))
@@
   (segment (start 134.527868 128.23715) (end 136.781474 125.983544) (width 0.381) (layer B.Cu) (net 107))
   (segment (start 117.268879 151.308879) (end 133.915685 151.308879) (width 0.381) (layer B.Cu) (net 107))
+  (segment (start 114.86 147.697919) (end 115.1 147.457919) (width 0.381) (layer B.Cu) (net 107))
+  (segment (start 114.86 148.9) (end 114.86 147.697919) (width 0.381) (layer B.Cu) (net 107))
+  (segment (start 115.1 147.457919) (end 115.1 144.8) (width 0.381) (layer B.Cu) (net 107))
   (segment (start 136.30015 124.821522) (end 169.243497 124.821522) (width 0.381) (layer B.Cu) (net 108))
   (segment (start 119.8 149.2) (end 120.740501 150.140501) (width 0.381) (layer B.Cu) (net 108))
@@
   (segment (start 174.327041 119.737977) (end 205.237977 119.737977) (width 0.381) (layer B.Cu) (net 108))
   (segment (start 120.740501 150.140501) (end 131.262401 150.140501) (width 0.381) (layer B.Cu) (net 108))
+  (segment (start 119.94 148.9) (end 119.94 144.66) (width 0.381) (layer B.Cu) (net 108))
+  (segment (start 119.94 144.66) (end 120 144.6) (width 0.381) (layer B.Cu) (net 108))
   (segment (start 212.3 114) (end 211.109499 115.190501) (width 0.381) (layer F.Cu) (net 109))
   (segment (start 211.109499 115.190501) (end 199.237978 115.190501) (width 0.381) (layer F.Cu) (net 109))
@@
   (segment (start 109.332923 153.632923) (end 134.878335 153.632923) (width 0.381) (layer B.Cu) (net 111))
   (segment (start 136.851912 151.659347) (end 136.851912 129.199798) (width 0.381) (layer B.Cu) (net 111))
-  (via (at 185.9 124.3) (size 0.8) (drill 0.4) (layers F.Cu B.Cu) (net 112))
-  (segment (start 229.409499 133.362559) (end 229.409499 136.309499) (width 0.381) (layer B.Cu) (net 105))
-  (segment (start 229.5 133.272058) (end 229.409499 133.362559) (width 0.381) (layer B.Cu) (net 105))
-  (segment (start 229.5 124.75137) (end 229.5 133.272058) (width 0.381) (layer B.Cu) (net 105))
-  (segment (start 228.28 122.4) (end 228.28 123.53137) (width 0.381) (layer B.Cu) (net 105))
-  (segment (start 228.28 123.53137) (end 229.5 124.75137) (width 0.381) (layer B.Cu) (net 105))
-  (segment (start 229.409499 136.309499) (end 229.5 136.4) (width 0.381) (layer B.Cu) (net 105))
-  (segment (start 114.86 147.697919) (end 115.1 147.457919) (width 0.381) (layer B.Cu) (net 107))
-  (segment (start 114.86 148.9) (end 114.86 147.697919) (width 0.381) (layer B.Cu) (net 107))
-  (segment (start 115.1 147.457919) (end 115.1 144.8) (width 0.381) (layer B.Cu) (net 107))
-  (segment (start 119.94 148.9) (end 119.94 144.66) (width 0.381) (layer B.Cu) (net 108))
-  (segment (start 119.94 144.66) (end 120 144.6) (width 0.381) (layer B.Cu) (net 108))
   (segment (start 234.7 118.2) (end 235.8 119.3) (width 0.381) (layer F.Cu) (net 111))
   (segment (start 234.7 109.575956) (end 234.7 118.2) (width 0.381) (layer F.Cu) (net 111))
@@
   (segment (start 104.7 148.9) (end 104.7 144.9) (width 0.381) (layer B.Cu) (net 111))
   (segment (start 104.7 144.9) (end 105 144.6) (width 0.381) (layer B.Cu) (net 111))
+  (via (at 185.9 124.3) (size 0.8) (drill 0.4) (layers F.Cu B.Cu) (net 112))
   (segment (start 137.262798 127.145566) (end 170.206145 127.145566) (width 0.381) (layer B.Cu) (net 112))
   (segment (start 170.206145 127.145566) (end 175.05171 122.3) (width 0.381) (layer B.Cu) (net 112))
